Commit message: Update prius.urdf

File: urdf/prius.urdf (robot description, URDF)
Before this commit: robot prius, 28 links, 27 joints
Links:
- link chassis: geometry collision box size=1.168381 1.654253 0.272347; collision box size=1.267845 1.116344 0.244286
- link front_left_wheel: geometry collision sphere radius=0.31265; visual mesh filename=models/wheel.obj scale=0.01 0.01 0.01
- link front_right_wheel: geometry collision sphere radius=0.31265; visual mesh filename=models/wheel.obj scale=0.01 0.01 0.01
- link rear_left_wheel: geometry collision sphere radius=0.31265; visual mesh filename=models/wheel.obj scale=0.01 0.01 0.01
- link rear_right_wheel: geometry collision sphere radius=0.31265; visual mesh filename=models/wheel.obj scale=0.01 0.01 0.01
- link steering_wheel: geometry visual mesh filename=models/steering_wheel.obj scale=0.01 0.01 0.01

Commit message: Update prius.urdf

File: urdf/prius.urdf (robot description, URDF)
Before this commit: robot prius, 9 links, 8 joints
Joints:
- joint front_left_steer_joint: limit lower=-0.8727 upper=0.8727 effort=10000000 velocity=1000000 -> (none)
- joint front_right_steer_joint: limit lower=-0.8727 upper=0.8727 effort=10000000 velocity=1000000 -> (none)
- joint steering_joint: limit lower=-7.85 upper=7.85 effort=10000000 velocity=1000000 -> (none)
